File: hardware/imspi8080.kicad_sch (KiCad schematic)
At the start: 85 parts, among them J1 USB_C_Receptacle_USB2.0_16P, J2 USB_C_Receptacle_USB2.0_16P, J3 Conn_01x10_Pin, J4 Conn_01x06_Pin, J5 Conn_01x03_Pin, SW1 SW_Push, SW2 SW_Push, U1 RP2040, U2 W25Q128JVS, U3 TLC5947DAP, U4 TLC5947DAP, U5 74HC165, U6 74HC165, U7 Micro_SD_Card, U8 AMS1117-3.3, U9 AMS1117-3.3, Y1 12MHz

Commit message: rev6 (wip): RP2350A netlist + schematic + pre-route board
Netlist surgery: U1 -> RP2350A (QFN-60-1EP 7x7 thermal-vias) with full pin
remap per REV6-PLAN.md; new L1 2.2uH (Bourns SRU5016 fp) wiring VREG_LX
(U1-48) to VREG_FB=VCORE; +3V3 also feeds VREG_AVDD/VIN + ADC_AVDD +
USB_OTP_VDD + QSPI_IOVDD; DVDD pins 6/23/39 on VCORE. Schematic regen
(gen_schematic.py) round-trip verified: every source net matches the export.

Board copy imspi8080_rev6.kicad_pcb: U1 footprint swapped at same pos/orient
(7x7 body), pads remapped, D1-D28 shifted -0.075mm to switch-pad columns,
L1 placed (138.713,86.854) r180, MCU-cluster + LED nets ripped (1166 trks /
105 vias). min through-drill relaxed 0.25->0.20mm for thermal vias. DRC:
110 cosmetic warnings, 187 unconnected awaiting autoroute (freerouting
running).

Also documented: rev5 firmware config.h was stale (HC chain on GPIO 7/8/9
per board, header said 10/11/12) - rev6 firmware fixes this for real.
Parts:
- added U1: RP2350A, Package_DFN_QFN:QFN-60-1EP_7x7mm_P0.4mm_EP3.4x3.4mm_ThermalVias, symbol MCU_RaspberryPi:RP2350A
- L1: renamed from R1; value 5.1k -> 2.2uH; footprint Resistor_SMD:R_0402_1005Metric -> Inductor_SMD:L_Bourns-SRU5016_5.2x5.2mm; symbol Device:R -> Device:L
- R16: renamed from SW1; value SW_Push -> 10k; footprint Button_Switch_SMD:SW_Push_1P1T_NO_CK_KMR2 -> Resistor_SMD:R_0402_1005Metric; symbol Switch:SW_Push -> Device:R
- R4: renamed from R5; value 27 -> 5.1k
- R6: renamed from R7; value 2.4k -> 27
- R8: renamed from R9; value 10k -> 2.4k
- SW2: renamed from U1; value RP2040 -> SW_Push; footprint Package_DFN_QFN:QFN-56-1EP_7x7mm_P0.4mm_EP3.2x3.2mm -> Button_Switch_SMD:SW_Push_1P1T_NO_CK_KMR2; symbol MCU_RaspberryPi:RP2040 -> Switch:SW_Push
- renumbered R2 to R1, R11 to R10, R12 to R11, R13 to R12, R14 to R13, R15 to R14, R16 to R15, R3 to R2, R4 to R3, R6 to R5, R8 to R7, R10 to R9, SW2 to SW1
Connections:
- net +3V3: now also R16.1, U1.1 (IOVDD), U1.11 (IOVDD), U1.20 (IOVDD), U1.30 (IOVDD), U1.38 (IOVDD), U1.44 (ADC_AVDD), U1.45 (IOVDD), U1.46 (VREG_AVDD), U1.49 (VREG_VIN), U1.53 (USB_OTP_VDD), U1.54 (QSPI_IOVDD); no longer R8.1, SW2.1 (IOVDD), SW2.10 (IOVDD), SW2.22 (IOVDD), SW2.33 (IOVDD), SW2.42 (IOVDD), SW2.43 (ADC_AVDD), SW2.44 (VREG_VIN), SW2.48 (USB_VDD), SW2.49 (IOVDD)
- net CMD0: now also R13.2; no longer R12.2
- net CMD1: now also R14.2; no longer R13.2
- net CMD2: now also R15.2; no longer R14.2
- net CMD3: now also R16.2; no longer R15.2
- net GND: now also R4.2, R8.2, SW2.2, U1.47 (VREG_PGND), U1.61 (GND); no longer L1.2, R16.2, R6.2, SW2.19 (TESTEN), SW2.57 (GND)
- net HC_CLK: now also U1.12 (GPIO8); no longer SW2.11 (GPIO8)
- net HC_PLOAD: now also U1.9 (GPIO6); no longer SW2.9 (GPIO7)
- net HC_QH: now also U1.13 (GPIO9); no longer SW2.12 (GPIO9)
- net N$1: now also U1.24 (SWCLK); no longer SW2.24 (SWCLK)
- net N$10: now also R8.1; no longer R7.1
- net N$2: now also U1.25 (SWDIO); no longer SW2.25 (SWDIO)
- net N$3: now also R1.1; no longer L1.1
- net N$39: now also R11.2; no longer R10.2
- net N$4: now also R2.1; no longer R1.1
- net N$40: now also R12.2; no longer R11.2
- net N$5: now also R3.1; no longer R2.1
- net N$6: now also R4.1; no longer R3.1
- net N$7: now also R5.2, U1.52 (USB_DP); no longer R4.2, SW2.47 (USB_DP)
- net N$8: now also R6.2, U1.51 (USB_DM); no longer R5.2, SW2.46 (USB_DM)
- net N$9: now also R7.1; no longer R6.1
- net QSPI_SCLK: now also U1.56 (QSPI_SCLK); no longer SW2.52 (QSPI_SCLK)
- net QSPI_SD0: now also U1.57 (QSPI_SD0); no longer SW2.53 (QSPI_SD0)
- net QSPI_SD1: now also U1.59 (QSPI_SD1); no longer SW2.55 (QSPI_SD1)
- net QSPI_SD2: now also U1.58 (QSPI_SD2); no longer SW2.54 (QSPI_SD2)
- net QSPI_SD3: now also U1.55 (QSPI_SD3); no longer SW2.51 (QSPI_SD3)
- net QSPI_SS: now also SW1.1, U1.60 (~{QSPI_SS}); no longer R16.1, SW2.56 (~{QSPI_SS})
- net RUN: now also SW2.1, U1.26 (RUN); no longer SW1.1, SW2.26 (RUN)
- net SD_CS: now also R9.2, U1.17 (GPIO13); no longer R8.2, SW2.16 (GPIO13)
- net SD_MISO: now also R10.2, U1.16 (GPIO12); no longer R9.2, SW2.15 (GPIO12)
- net SD_MOSI: now also U1.15 (GPIO11); no longer SW2.14 (GPIO11)
- net SD_SCK: now also U1.14 (GPIO10); no longer SW2.13 (GPIO10)
- net TLC_BLANK: now also U1.8 (GPIO5); no longer SW2.7 (GPIO5)
- net TLC_SCLK: now also U1.4 (GPIO2); no longer SW2.4 (GPIO2)
- net TLC_SIN: now also U1.5 (GPIO3); no longer SW2.5 (GPIO3)
- net TLC_XLAT: now also U1.7 (GPIO4); no longer SW2.6 (GPIO4)
- net USB_DM_CONN: now also R6.1; no longer R5.1
- net USB_DP_CONN: now also R5.1; no longer R4.1
- net VCORE: now also L1.2, U1.23 (DVDD), U1.39 (DVDD), U1.50 (VREG_FB), U1.6 (DVDD); no longer SW2.23 (DVDD), SW2.45 (VREG_VOUT), SW2.50 (DVDD)
- net XIN: now also U1.21 (XIN); no longer SW2.20 (XIN)
- net XOUT: now also U1.22 (XOUT); no longer SW2.21 (XOUT)
- new net VREG_LX: L1.1, U1.48 (VREG_LX)
