File: hardware/imspi8080_rev6.kicad_pcb (KiCad board)
At the start: 4 copper layers, 204 x 112 mm, 126 parts, among them J1 USB_C_Receptacle_USB2.0_16P, J2 USB_C_Receptacle_USB2.0_16P, J5 Conn_01x03_Pin, SW1 SW_Push, SW2 SW_Push, U1 RP2350A, U2 W25Q128JVS, U3 TLC5947DAP, U4 TLC5947DAP, U5 74HC165, U6 74HC165, U7 Micro_SD_Card, U8 AMS1117-3.3, U9 AMS1117-3.3, Y1 12MHz

Commit message: rev6 (wip): post-route baseline (SES import + GND pour, one zone)
Routing:
- net +3V3: track 0.00 -> 584.3 mm, vias 0 -> 8
- net +3V3_LED: track 0.00 -> 449.7 mm, vias 0 -> 2
- net HC_CLK: track 0.00 -> 127.3 mm, vias 0 -> 3
- net TLC_SCLK: track 0.00 -> 125.7 mm, vias 0 -> 2
- net HC_PLOAD: track 0.00 -> 125.3 mm, vias 0 -> 3
- net TLC_XLAT: track 0.00 -> 120.3 mm, vias 0 -> 2
- net TLC_BLANK: track 0.00 -> 119.4 mm, vias 0 -> 3
- net SD_MISO: track 0.00 -> 117.7 mm, vias 0 -> 2
- net SD_CS: track 0.00 -> 106.4 mm, vias 0 -> 2
- net SD_SCK: track 0.00 -> 102.1 mm, vias 0 -> 2
- net SD_MOSI: track 0.00 -> 102.0 mm, vias 0 -> 2
- net HC_QH: track 0.00 -> 76.8 mm, vias 0 -> 2
- net N$27: track 0.00 -> 69.9 mm, vias 0 -> 2
- net N$2: track 0.00 -> 66.9 mm, vias 0 -> 1
- net N$1: track 0.00 -> 66.8 mm, vias 0 -> 1
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
Commit message: rev6: complete — fully routed RP2350A board, fab package, clean checks
Board: DRC 110 (all cosmetic: 80 back-silk text, 24 silk overlap,
6 stub warnings), 0 errors. check_opens.py: every net a single copper
island — the two rev5 assembly wires (HC_QH, TLC_SCLK) are routed, the
allow-list is empty for rev6. Fixed along the way: freerouting GND
skip root-caused (KiCad DSN emits the GND zone as a Specctra plane;
fix = no zones before export_dsn), duplicate via + zero-length stubs
cleaned, checker now reads pads' full copper layer set (GetLayer lies
for multi-layer pads).

Fab package fab-rev6/: gerbers (14), drill PTH/NPTH, gbrjob, BOM
csv+xlsx (96 rows: U1=RP2350A C42411118 in stock at JLCPCB, +L1 2.2uH
VREG inductor), CPL (96, BOM==CPL verified), README with RP2350
bring-up checklist (flash-list + crystal cap verification, no
assembly wires).
Routing:
- net GND: track 40.5 -> 793.5 mm, vias 22 -> 24
- net VCORE: track 37.7 -> 38.3 mm
- net HC_PLOAD: track 125.3 -> 125.9 mm
